File: rbe-tmag5273/rbe-tmag5273.kicad_sch (KiCad schematic)
At the start: 0 parts

Commit message: Add new KiCad project rbe-tmag5273
This commit introduces a new KiCad project for the TMAG5273A2QDBVR component.

Includes:
- Schematic and PCB layout files.
- Custom footprint and 3D model for TMAG5273A2QDBVR.
- KiCad project configuration and library tables.
- A generated interactive BOM (ibom.html) for easy review.
Parts:
- added C1: 100nF, Capacitor_SMD:C_0603_1608Metric, symbol Device:C
- added D1: LED, LED_SMD:LED_0603_1608Metric, symbol Device:LED
- added H1, H2, H3, H4: MountingHole_Pad, MountingHole:MountingHole_3.2mm_M3_Pad, symbol Mechanical:MountingHole_Pad
- added J1, J2: Conn_01x04, Connector_PinHeader_2.54mm:PinHeader_1x04_P2.54mm_Vertical, symbol Connector_Generic:Conn_01x04
- added J3, J4: Conn_01x04_MountingPin, Connector_JST:JST_SH_SM04B-SRSS-TB_1x04-1MP_P1.00mm_Horizontal, symbol Connector_Generic_MountingPin:Conn_01x04_MountingPin
- added R1, R2: 2.2k, Resistor_SMD:R_0603_1608Metric, symbol Device:R
- added R3: R, Resistor_SMD:R_0603_1608Metric, symbol Device:R
- added R4: 10k, Resistor_SMD:R_0603_1608Metric, symbol Device:R
- added U1: TMAG5273A2QDBVR, TMAG5273A2QDBVR:SOT95P280X140-6N, symbol TMAG5273A2QDBVR:TMAG5273A2QDBVR
Connections:
- new net: D1.2 (A), R3.2
- new net +3V3: C1.1, J1.2 (Pin_2), J2.3 (Pin_3), J3.2 (Pin_2), J4.2 (Pin_2), R1.1, R2.1, R3.1, R4.1, U1.4 (VCC)
- new net GND: C1.2, D1.1 (K), H1.1, H2.1, H3.1, H4.1, J1.1 (Pin_1), J2.1 (Pin_1), J2.2 (Pin_2), J3.1 (Pin_1), J3.MP (MountPin), J4.1 (Pin_1), J4.MP (MountPin), U1.2 (GND), U1.3 (TEST)
- new net SCL: J1.4 (Pin_4), J3.4 (Pin_4), J4.4 (Pin_4), R2.2, U1.1 (SCL)
- new net SDA: J1.3 (Pin_3), J3.3 (Pin_3), J4.3 (Pin_3), R1.2, U1.6 (SDA)
- new net ~{INT}: J2.4 (Pin_4), R4.2, U1.5 (~{INT})
Other:
- company: (none) -> PT Reka Bentuk Elektronika
- title: (none) -> RBE TMAG5273
